File: Logic_power.kicad_sch (KiCad schematic)
At the start: 13 parts, among them U8 TPS5430DDA, U9 XC6206P332MR-G

Commit message: Parts layout finish
Parts:
- D19: LCSC C509937 -> C22466347
Changed lines of the file:
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@@
       (project "schematic_PWR"
         (path "/f4729e9b-1fa3-4d29-bc6f-94f153418360/5172fa46-aba7-443b-901c-ede9474f0ff0"
-          (reference "C1") (unit 1)
+          (reference "C30") (unit 1)
         )
       )
@@
       (project "schematic_PWR"
         (path "/f4729e9b-1fa3-4d29-bc6f-94f153418360/5172fa46-aba7-443b-901c-ede9474f0ff0"
-          (reference "C55") (unit 1)
+          (reference "C29") (unit 1)
         )
       )
@@
       (project "schematic_PWR"
         (path "/f4729e9b-1fa3-4d29-bc6f-94f153418360/5172fa46-aba7-443b-901c-ede9474f0ff0"
-          (reference "R4") (unit 1)
+          (reference "R21") (unit 1)
         )
       )
@@
       (project "schematic_PWR"
         (path "/f4729e9b-1fa3-4d29-bc6f-94f153418360/5172fa46-aba7-443b-901c-ede9474f0ff0"
-          (reference "D18") (unit 1)
+          (reference "D7") (unit 1)
         )
       )
@@
       (project "schematic_PWR"
         (path "/f4729e9b-1fa3-4d29-bc6f-94f153418360/5172fa46-aba7-443b-901c-ede9474f0ff0"
-          (reference "U9") (unit 1)
+          (reference "U5") (unit 1)
         )
       )
@@
       (project "schematic_PWR"
         (path "/f4729e9b-1fa3-4d29-bc6f-94f153418360/5172fa46-aba7-443b-901c-ede9474f0ff0"
-          (reference "R1") (unit 1)
+          (reference "R20") (unit 1)
         )
       )
@@
       (effects (font (size 1.27 1.27)) hide)
     )
-    (property "LCSC" "C509937" (at 165.1 55.88 0)
+    (property "LCSC" "C22466347" (at 165.1 55.88 0)
       (effects (font (size 1.27 1.27)) hide)
     )
@@
       (project "schematic_PWR"
         (path "/f4729e9b-1fa3-4d29-bc6f-94f153418360/5172fa46-aba7-443b-901c-ede9474f0ff0"
-          (reference "D19") (unit 1)
+          (reference "D8") (unit 1)
         )
       )
@@
       (project "schematic_PWR"
         (path "/f4729e9b-1fa3-4d29-bc6f-94f153418360/5172fa46-aba7-443b-901c-ede9474f0ff0"
-          (reference "C58") (unit 1)
+          (reference "C32") (unit 1)
         )
       )
@@
       (project "schematic_PWR"
         (path "/f4729e9b-1fa3-4d29-bc6f-94f153418360/5172fa46-aba7-443b-901c-ede9474f0ff0"
-          (reference "C57") (unit 1)
+          (reference "C31") (unit 1)
         )
       )
@@
       (project "schematic_PWR"
         (path "/f4729e9b-1fa3-4d29-bc6f-94f153418360/5172fa46-aba7-443b-901c-ede9474f0ff0"
-          (reference "U8") (unit 1)
+          (reference "U4") (unit 1)
         )
       )
@@
       (project "schematic_PWR"
         (path "/f4729e9b-1fa3-4d29-bc6f-94f153418360/5172fa46-aba7-443b-901c-ede9474f0ff0"
-          (reference "C54") (unit 1)
+          (reference "C28") (unit 1)
         )
       )
@@
       (project "schematic_PWR"
         (path "/f4729e9b-1fa3-4d29-bc6f-94f153418360/5172fa46-aba7-443b-901c-ede9474f0ff0"
-          (reference "R1") (unit 1)
-        )
-      )
+          (reference "R19") (unit 1)
+        )
+      )
