File: EMS.kicad_sch (KiCad schematic)
At the start: 14 parts, among them J12 Conn_01x02, J13 Conn_01x02, Q4 Q_NMOS_GSD, Q5 Q_PMOS_GSD, Q6 Q_NMOS_GSD

Commit message: Parts layout finish
Parts:
- R13, R14, R15, R16, R17, R18, R22: footprint Resistor_SMD:R_0603_1608Metric_Pad0.98x0.95mm_HandSolder -> Resistor_SMD:R_0402_1005Metric
Other:
- note removed: "最大伝達遅延 11.757us"
- note removed: "最大伝達遅延 16.257us"
- note removed: "遅延 0.087us"
- note removed: "遅延 11.67us"
- note removed: "遅延 4.5us"
Changed lines of the file:
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@@
     (stroke (width 0) (type default))
-  )
-  (text "遅延 0.087us" (at 116.84 109.22 0)
-    (effects (font (size 1.27 1.27)) (justify left bottom))
-  )
-  (text "最大伝達遅延 16.257us" (at 229.87 99.06 0)
-    (effects (font (size 1.27 1.27)) (justify left bottom))
-  )
-  (text "遅延 4.5us" (at 208.28 106.68 0)
-    (effects (font (size 1.27 1.27)) (justify left bottom))
-  )
-  (text "最大伝達遅延 11.757us" (at 187.96 53.34 0)
-    (effects (font (size 1.27 1.27)) (justify left bottom))
-  )
-  (text "遅延 11.67us" (at 96.52 49.53 0)
-    (effects (font (size 1.27 1.27)) (justify left bottom))
   )
   (hierarchical_label "Relay_Signal_IN" (shape input) (at 59.69 58.42 180) (fields_autoplaced)
@@
       (project "schematic_PWR"
         (path "/f4729e9b-1fa3-4d29-bc6f-94f153418360/ac952d49-c6b8-4a25-9eb5-040b6bb0e6d0"
-          (reference "J12") (unit 1)
+          (reference "J13") (unit 1)
         )
       )
@@
       (effects (font (size 1.27 1.27)))
     )
-    (property "Footprint" "Resistor_SMD:R_0603_1608Metric_Pad0.98x0.95mm_HandSolder" (at 186.69 97.282 90)
+    (property "Footprint" "Resistor_SMD:R_0402_1005Metric" (at 186.69 97.282 90)
       (effects (font (size 1.27 1.27)) hide)
     )
@@
       (project "schematic_PWR"
         (path "/f4729e9b-1fa3-4d29-bc6f-94f153418360/ac952d49-c6b8-4a25-9eb5-040b6bb0e6d0"
-          (reference "R16") (unit 1)
+          (reference "R29") (unit 1)
         )
       )
@@
       (project "schematic_PWR"
         (path "/f4729e9b-1fa3-4d29-bc6f-94f153418360/ac952d49-c6b8-4a25-9eb5-040b6bb0e6d0"
-          (reference "Q4") (unit 1)
+          (reference "Q6") (unit 1)
         )
       )
@@
       (project "schematic_PWR"
         (path "/f4729e9b-1fa3-4d29-bc6f-94f153418360/ac952d49-c6b8-4a25-9eb5-040b6bb0e6d0"
-          (reference "J13") (unit 1)
+          (reference "J14") (unit 1)
         )
       )
@@
       (effects (font (size 1.27 1.27)) (justify right))
     )
-    (property "Footprint" "Resistor_SMD:R_0603_1608Metric_Pad0.98x0.95mm_HandSolder" (at 109.982 78.74 90)
+    (property "Footprint" "Resistor_SMD:R_0402_1005Metric" (at 109.982 78.74 90)
       (effects (font (size 1.27 1.27)) hide)
     )
@@
       (project "schematic_PWR"
         (path "/f4729e9b-1fa3-4d29-bc6f-94f153418360/ac952d49-c6b8-4a25-9eb5-040b6bb0e6d0"
-          (reference "R15") (unit 1)
+          (reference "R28") (unit 1)
         )
       )
@@
       (effects (font (size 1.27 1.27)))
     )
-    (property "Footprint" "Resistor_SMD:R_0603_1608Metric_Pad0.98x0.95mm_HandSolder" (at 96.52 96.012 90)
+    (property "Footprint" "Resistor_SMD:R_0402_1005Metric" (at 96.52 96.012 90)
       (effects (font (size 1.27 1.27)) hide)
     )
@@
       (project "schematic_PWR"
         (path "/f4729e9b-1fa3-4d29-bc6f-94f153418360/ac952d49-c6b8-4a25-9eb5-040b6bb0e6d0"
-          (reference "R13") (unit 1)
+          (reference "R25") (unit 1)
         )
       )
@@
       (effects (font (size 1.27 1.27)) (justify right))
     )
-    (property "Footprint" "Resistor_SMD:R_0603_1608Metric_Pad0.98x0.95mm_HandSolder" (at 96.012 66.04 90)
+    (property "Footprint" "Resistor_SMD:R_0402_1005Metric" (at 96.012 66.04 90)
       (effects (font (size 1.27 1.27)) hide)
     )
@@
       (project "schematic_PWR"
         (path "/f4729e9b-1fa3-4d29-bc6f-94f153418360/ac952d49-c6b8-4a25-9eb5-040b6bb0e6d0"
-          (reference "R22") (unit 1)
+          (reference "R26") (unit 1)
         )
       )
@@
       (project "schematic_PWR"
         (path "/f4729e9b-1fa3-4d29-bc6f-94f153418360/ac952d49-c6b8-4a25-9eb5-040b6bb0e6d0"
-          (reference "Q5") (unit 1)
+          (reference "Q7") (unit 1)
         )
       )
@@
       (project "schematic_PWR"
         (path "/f4729e9b-1fa3-4d29-bc6f-94f153418360/ac952d49-c6b8-4a25-9eb5-040b6bb0e6d0"
-          (reference "Q6") (unit 1)
+          (reference "Q8") (unit 1)
         )
       )
@@
       (effects (font (size 1.27 1.27)) (justify right))
     )
-    (property "Footprint" "Resistor_SMD:R_0603_1608Metric_Pad0.98x0.95mm_HandSolder" (at 194.818 105.41 90)
+    (property "Footprint" "Resistor_SMD:R_0402_1005Metric" (at 194.818 105.41 90)
       (effects (font (size 1.27 1.27)) hide)
     )
@@
       (project "schematic_PWR"
         (path "/f4729e9b-1fa3-4d29-bc6f-94f153418360/ac952d49-c6b8-4a25-9eb5-040b6bb0e6d0"
-          (reference "R17") (unit 1)
+          (reference "R30") (unit 1)
         )
       )
@@
       (project "schematic_PWR"
         (path "/f4729e9b-1fa3-4d29-bc6f-94f153418360/ac952d49-c6b8-4a25-9eb5-040b6bb0e6d0"
-          (reference "JP1") (unit 1)
+          (reference "JP3") (unit 1)
         )
       )
@@
       (project "schematic_PWR"
         (path "/f4729e9b-1fa3-4d29-bc6f-94f153418360/ac952d49-c6b8-4a25-9eb5-040b6bb0e6d0"
-          (reference "JP1") (unit 1)
+          (reference "JP2") (unit 1)
         )
       )
@@
       (effects (font (size 1.27 1.27)) (justify right))
     )
-    (property "Footprint" "Resistor_SMD:R_0603_1608Metric_Pad0.98x0.95mm_HandSolder" (at 203.708 85.09 90)
+    (property "Footprint" "Resistor_SMD:R_0402_1005Metric" (at 203.708 85.09 90)
       (effects (font (size 1.27 1.27)) hide)
     )
@@
       (project "schematic_PWR"
         (path "/f4729e9b-1fa3-4d29-bc6f-94f153418360/ac952d49-c6b8-4a25-9eb5-040b6bb0e6d0"
-          (reference "R18") (unit 1)
+          (reference "R31") (unit 1)
         )
       )
@@
       (effects (font (size 1.27 1.27)) (justify right))
     )
-    (property "Footprint" "Resistor_SMD:R_0603_1608Metric_Pad0.98x0.95mm_HandSolder" (at 104.648 104.14 90)
+    (property "Footprint" "Resistor_SMD:R_0402_1005Metric" (at 104.648 104.14 90)
       (effects (font (size 1.27 1.27)) hide)
     )
@@
       (project "schematic_PWR"
         (path "/f4729e9b-1fa3-4d29-bc6f-94f153418360/ac952d49-c6b8-4a25-9eb5-040b6bb0e6d0"
-          (reference "R14") (unit 1)
-        )
-      )
+          (reference "R27") (unit 1)
+        )
+      )

Commit message: update art work
Parts:
- J12, J13: footprint Connector_JST:JST_XA_B02B-XASK-1_1x02_P2.50mm_Vertical -> Connector_JST:JST_XA_S02B-XASK-1_1x02_P2.50mm_Horizontal
Changed lines of the file:
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@@
       (effects (font (size 1.27 1.27)))
     )
-    (property "Footprint" "Connector_JST:JST_XA_B02B-XASK-1_1x02_P2.50mm_Vertical" (at 124.46 66.04 0)
+    (property "Footprint" "Connector_JST:JST_XA_S02B-XASK-1_1x02_P2.50mm_Horizontal" (at 124.46 66.04 0)
       (effects (font (size 1.27 1.27)) hide)
     )
@@
       (effects (font (size 1.27 1.27)))
     )
-    (property "Footprint" "Connector_JST:JST_XA_B02B-XASK-1_1x02_P2.50mm_Vertical" (at 137.16 66.04 0)
+    (property "Footprint" "Connector_JST:JST_XA_S02B-XASK-1_1x02_P2.50mm_Horizontal" (at 137.16 66.04 0)
       (effects (font (size 1.27 1.27)) hide)
     )

Commit message: アートワークのほとんど終わり
Parts:
- Q4, Q6: LCSC (none) -> C7420346
- Q5: LCSC (none) -> C15127
- R13, R16: LCSC (none) -> C25076
- R14, R15, R17, R18, R22: LCSC (none) -> C25744
Changed lines of the file:
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@@
+      (effects (font (size 1.27 1.27)) hide)
+    )
+    (property "LCSC" "C25076" (at 186.69 99.06 0)
       (effects (font (size 1.27 1.27)) hide)
     )
@@
       (effects (font (size 1.27 1.27)) hide)
     )
+    (property "LCSC" "C7420346" (at 109.22 97.79 0)
+      (effects (font (size 1.27 1.27)) hide)
+    )
     (pin "1")
     (pin "3")
@@
       (effects (font (size 1.27 1.27)) hide)
     )
+    (property "LCSC" "C25744" (at 111.76 78.74 0)
+      (effects (font (size 1.27 1.27)) hide)
+    )
     (pin "1")
     (pin "2")
@@
       (effects (font (size 1.27 1.27)) hide)
     )
+    (property "LCSC" "C25076" (at 96.52 97.79 0)
+      (effects (font (size 1.27 1.27)) hide)
+    )
     (pin "2")
     (pin "1")
@@
       (effects (font (size 1.27 1.27)) hide)
     )
+    (property "LCSC" "C25744" (at 97.79 66.04 0)
+      (effects (font (size 1.27 1.27)) hide)
+    )
     (pin "1")
     (pin "2")
@@
     )
     (property "name" "" (at 111.76 60.96 0)
+      (effects (font (size 1.27 1.27)) hide)
+    )
+    (property "LCSC" "C15127" (at 111.76 60.96 0)
       (effects (font (size 1.27 1.27)) hide)
     )
@@
       (effects (font (size 1.27 1.27)) hide)
     )
+    (property "LCSC" "C7420346" (at 199.39 99.06 0)
+      (effects (font (size 1.27 1.27)) hide)
+    )
     (pin "1")
     (pin "3")
@@
     )
     (property "name" "" (at 193.04 105.41 0)
+      (effects (font (size 1.27 1.27)) hide)
+    )
+    (property "LCSC" "C25744" (at 193.04 105.41 0)
       (effects (font (size 1.27 1.27)) hide)
     )
@@
       (effects (font (size 1.27 1.27)) hide)
     )
+    (property "LCSC" "C25744" (at 201.93 85.09 0)
+      (effects (font (size 1.27 1.27)) hide)
+    )
     (pin "1")
     (pin "2")
@@
       (effects (font (size 1.27 1.27)) hide)
     )
+    (property "LCSC" "C25744" (at 102.87 104.14 0)
+      (effects (font (size 1.27 1.27)) hide)
+    )
