File: Power_relay.kicad_sch (KiCad schematic)
At the start: 8 parts, among them K1 HE1AN-W-DC12V-Y6, Q5 Q_NMOS_GSD

Commit message: Parts layout finish
Parts:
- D10: renamed from D5; footprint (none) -> Diode_SMD:D_SOD-123F; LCSC (none) -> C22466347
- D11: renamed from D6; footprint (none) -> Diode_SMD:D_SOD-123F
- Q5: footprint (none) -> Package_TO_SOT_SMD:SOT-23
- R22: renamed from R18; footprint (none) -> Resistor_SMD:R_0402_1005Metric
- R23: renamed from R17; footprint (none) -> Resistor_SMD:R_0402_1005Metric
- R24: renamed from R16; footprint (none) -> Resistor_SMD:R_0402_1005Metric
- renumbered D7 to D9
Connections:
- net Coil_power: now also K1.4; no longer K1.3
- net Main_power_IN: now also K1.1; no longer K1.2
- net Main_power_OUT: now also K1.2; no longer K1.1
- net at D11.1 (K), D9.1 (K), Q5.3 (D): now also K1.3; no longer K1.4
Changed lines of the file:
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@@
     (stroke (width 0) (type default))
   )
-  (wire (pts (xy 123.19 101.6) (xy 147.32 101.6))
+  (wire (pts (xy 125.73 101.6) (xy 147.32 101.6))
     (stroke (width 0) (type default))
   )
@@
     (stroke (width 0) (type default))
   )
+  (wire (pts (xy 96.52 81.28) (xy 96.52 76.2))
+    (stroke (width 0) (type default))
+  )
+  (wire (pts (xy 113.03 88.9) (xy 96.52 88.9))
+    (stroke (width 0) (type default))
+  )
+  (wire (pts (xy 125.73 86.36) (xy 125.73 101.6))
+    (stroke (width 0) (type default))
+  )
+  (wire (pts (xy 71.12 118.11) (xy 90.17 118.11))
+    (stroke (width 0) (type default))
+  )
+  (wire (pts (xy 101.6 132.08) (xy 113.03 132.08))
+    (stroke (width 0) (type default))
+  )
+  (wire (pts (xy 113.03 46.99) (xy 113.03 59.69))
+    (stroke (width 0) (type default))
+  )
   (wire (pts (xy 113.03 96.52) (xy 113.03 113.03))
     (stroke (width 0) (type default))
   )
-  (wire (pts (xy 96.52 81.28) (xy 96.52 76.2))
-    (stroke (width 0) (type default))
-  )
-  (wire (pts (xy 113.03 88.9) (xy 96.52 88.9))
-    (stroke (width 0) (type default))
-  )
-  (wire (pts (xy 71.12 118.11) (xy 90.17 118.11))
-    (stroke (width 0) (type default))
-  )
-  (wire (pts (xy 101.6 132.08) (xy 113.03 132.08))
-    (stroke (width 0) (type default))
-  )
-  (wire (pts (xy 113.03 46.99) (xy 113.03 59.69))
-    (stroke (width 0) (type default))
-  )
-  (wire (pts (xy 125.73 46.99) (xy 125.73 71.12))
+  (wire (pts (xy 123.19 46.99) (xy 123.19 71.12))
     (stroke (width 0) (type default))
   )
@@
   )
   (wire (pts (xy 101.6 118.11) (xy 101.6 120.65))
-    (stroke (width 0) (type default))
-  )
-  (wire (pts (xy 123.19 86.36) (xy 123.19 101.6))
     (stroke (width 0) (type default))
   )
@@
     (effects (font (size 1.27 1.27)) (justify left))
   )
-  (hierarchical_label "Main_power_IN" (shape input) (at 125.73 46.99 90) (fields_autoplaced)
+  (hierarchical_label "Main_power_IN" (shape input) (at 123.19 46.99 90) (fields_autoplaced)
     (effects (font (size 1.27 1.27)) (justify left))
   )
-  (symbol (lib_id "RDC_generic:HE1AN-W-DC12V-Y6") (at 118.11 87.63 0) (unit 1)
-    (in_bom yes) (on_board yes) (dnp no) (fields_autoplaced)
-    (property "Reference" "K1" (at 129.54 77.47 0)
-      (effects (font (size 1.27 1.27)) (justify left))
-    )
-    (property "Value" "HE1AN-W-DC12V-Y6" (at 129.54 80.01 0)
-      (effects (font (size 1.27 1.27)) (justify left))
-    )
-    (property "Footprint" "RDC_generic:HE1AN-W-DC12V-Y6" (at 118.11 88.9 0)
-      (effects (font (size 1.27 1.27)) hide)
-    )
-    (property "Datasheet" "" (at 118.11 87.63 0)
+  (symbol (lib_id "RDC_generic:HE1AN-W-DC12V-Y6") (at 118.11 69.85 0) (mirror x) (unit 1)
+    (in_bom yes) (on_board yes) (dnp no)
+    (property "Reference" "K1" (at 129.54 80.01 0)
+      (effects (font (size 1.27 1.27)) (justify left))
+    )
+    (property "Value" "HE1AN-W-DC12V-Y6" (at 129.54 77.47 0)
+      (effects (font (size 1.27 1.27)) (justify left))
+    )
+    (property "Footprint" "RDC_generic:HE1AN-W-DC12V-Y6" (at 118.11 68.58 0)
+      (effects (font (size 1.27 1.27)) hide)
+    )
+    (property "Datasheet" "" (at 118.11 69.85 0)
       (effects (font (size 1.27 1.27)) hide)
     )
@@
   (symbol (lib_id "Device:R") (at 101.6 124.46 0) (mirror y) (unit 1)
     (in_bom yes) (on_board yes) (dnp no) (fields_autoplaced)
-    (property "Reference" "R16" (at 104.14 123.19 0)
+    (property "Reference" "R24" (at 104.14 123.19 0)
       (effects (font (size 1.27 1.27)) (justify right))
     )
@@
       (effects (font (size 1.27 1.27)) (justify right))
     )
-    (property "Footprint" "" (at 103.378 124.46 90)
+    (property "Footprint" "Resistor_SMD:R_0402_1005Metric" (at 103.378 124.46 90)
       (effects (font (size 1.27 1.27)) hide)
     )
@@
       (project "schematic_PWR"
         (path "/f4729e9b-1fa3-4d29-bc6f-94f153418360/6caf726e-6749-4027-bb17-fb44ad15ad78"
-          (reference "R16") (unit 1)
+          (reference "R24") (unit 1)
         )
       )
@@
       (effects (font (size 1.27 1.27)) (justify left))
     )
-    (property "Footprint" "" (at 115.57 115.57 0)
+    (property "Footprint" "Package_TO_SOT_SMD:SOT-23" (at 115.57 115.57 0)
       (effects (font (size 1.27 1.27)) hide)
     )
@@
   (symbol (lib_id "Device:R") (at 93.98 118.11 90) (mirror x) (unit 1)
     (in_bom yes) (on_board yes) (dnp no) (fields_autoplaced)
-    (property "Reference" "R17" (at 93.98 111.76 90)
+    (property "Reference" "R23" (at 93.98 111.76 90)
       (effects (font (size 1.27 1.27)))
     )
@@
       (effects (font (size 1.27 1.27)))
     )
-    (property "Footprint" "" (at 93.98 116.332 90)
+    (property "Footprint" "Resistor_SMD:R_0402_1005Metric" (at 93.98 116.332 90)
       (effects (font (size 1.27 1.27)) hide)
     )
@@
       (project "schematic_PWR"
         (path "/f4729e9b-1fa3-4d29-bc6f-94f153418360/6caf726e-6749-4027-bb17-fb44ad15ad78"
-          (reference "R17") (unit 1)
+          (reference "R23") (unit 1)
         )
       )
@@
   (symbol (lib_id "Device:D_Zener") (at 96.52 85.09 270) (mirror x) (unit 1)
     (in_bom yes) (on_board yes) (dnp no) (fields_autoplaced)
-    (property "Reference" "D6" (at 93.98 83.82 90)
+    (property "Reference" "D11" (at 93.98 83.82 90)
       (effects (font (size 1.27 1.27)) (justify right))
     )
@@
       (effects (font (size 1.27 1.27)) (justify right))
     )
-    (property "Footprint" "" (at 96.52 85.09 0)
+    (property "Footprint" "Diode_SMD:D_SOD-123F" (at 96.52 85.09 0)
       (effects (font (size 1.27 1.27)) hide)
     )
@@
       (project "schematic_PWR"
         (path "/f4729e9b-1fa3-4d29-bc6f-94f153418360/6caf726e-6749-4027-bb17-fb44ad15ad78"
-          (reference "D6") (unit 1)
+          (reference "D11") (unit 1)
         )
       )
@@
   (symbol (lib_id "Device:LED") (at 74.93 81.28 270) (mirror x) (unit 1)
     (in_bom yes) (on_board yes) (dnp no) (fields_autoplaced)
-    (property "Reference" "D7" (at 71.12 81.5975 90)
+    (property "Reference" "D9" (at 71.12 81.5975 90)
       (effects (font (size 1.27 1.27)) (justify right))
     )
@@
       (project "schematic_PWR"
         (path "/f4729e9b-1fa3-4d29-bc6f-94f153418360/6caf726e-6749-4027-bb17-fb44ad15ad78"
-          (reference "D7") (unit 1)
+          (reference "D9") (unit 1)
         )
       )
@@
   (symbol (lib_id "Device:R") (at 74.93 72.39 0) (unit 1)
     (in_bom yes) (on_board yes) (dnp no) (fields_autoplaced)
-    (property "Reference" "R18" (at 72.39 71.12 0)
+    (property "Reference" "R22" (at 72.39 71.12 0)
       (effects (font (size 1.27 1.27)) (justify right))
     )
@@
       (effects (font (size 1.27 1.27)) (justify right))
     )
-    (property "Footprint" "" (at 73.152 72.39 90)
+    (property "Footprint" "Resistor_SMD:R_0402_1005Metric" (at 73.152 72.39 90)
       (effects (font (size 1.27 1.27)) hide)
     )
@@
       (project "schematic_PWR"
         (path "/f4729e9b-1fa3-4d29-bc6f-94f153418360/6caf726e-6749-4027-bb17-fb44ad15ad78"
-          (reference "R18") (unit 1)
+          (reference "R22") (unit 1)
         )
       )
@@
   (symbol (lib_id "Device:D_Schottky") (at 96.52 72.39 90) (mirror x) (unit 1)
     (in_bom yes) (on_board yes) (dnp no) (fields_autoplaced)
-    (property "Reference" "D5" (at 93.98 70.8025 90)
+    (property "Reference" "D10" (at 93.98 70.8025 90)
       (effects (font (size 1.27 1.27)) (justify left))
     )
@@
       (effects (font (size 1.27 1.27)) (justify left))
     )
-    (property "Footprint" "" (at 96.52 72.39 0)
+    (property "Footprint" "Diode_SMD:D_SOD-123F" (at 96.52 72.39 0)
       (effects (font (size 1.27 1.27)) hide)
     )
@@
       (effects (font (size 1.27 1.27)) hide)
     )
-    (pin "2")
-    (pin "1")
-    (instances
-      (project "schematic_PWR"
-        (path "/f4729e9b-1fa3-4d29-bc6f-94f153418360/6caf726e-6749-4027-bb17-fb44ad15ad78"
-          (reference "D5") (unit 1)
-        )
-      )
+    (property "LCSC" "C22466347" (at 96.52 72.39 0)
+      (effects (font (size 1.27 1.27)) hide)
+    )
+    (pin "2")
+    (pin "1")
+    (instances
+      (project "schematic_PWR"
+        (path "/f4729e9b-1fa3-4d29-bc6f-94f153418360/6caf726e-6749-4027-bb17-fb44ad15ad78"
+          (reference "D10") (unit 1)
+        )
+      )

Commit message: update art work
Parts:
- K1: footprint RDC_generic:HE1AN-W-DC12V-Y6 -> RDC_generic:HE1AN-W-DC12V-Y6+Y5
Changed lines of the file:
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@@
       (effects (font (size 1.27 1.27)) (justify left))
     )
-    (property "Footprint" "RDC_generic:HE1AN-W-DC12V-Y6" (at 118.11 68.58 0)
+    (property "Footprint" "RDC_generic:HE1AN-W-DC12V-Y6+Y5" (at 118.11 68.58 0)
       (effects (font (size 1.27 1.27)) hide)
     )

Commit message: アートワークのほとんど終わり
Parts:
- D10: value D_Schottky -> D; symbol Device:D_Schottky -> Device:D; LCSC C22466347 -> C18199085
- D11: footprint Diode_SMD:D_SOD-123F -> Diode_SMD:D_SMA; LCSC (none) -> C19077489
- D9: footprint LED_SMD:LED_0603_1608Metric_Pad1.05x0.95mm_HandSolder -> LED_SMD:LED_0603_1608Metric; LCSC (none) -> C2286
- Q5: LCSC (none) -> C7420346
- R22, R24: LCSC (none) -> C25744
- R23: LCSC (none) -> C25076
Changed lines of the file:
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@@
+      (effects (font (size 1.27 1.27)) hide)
+    )
+    (property "LCSC" "C25744" (at 101.6 124.46 0)
       (effects (font (size 1.27 1.27)) hide)
     )
@@
     )
     (property "Datasheet" "~" (at 110.49 118.11 0)
+      (effects (font (size 1.27 1.27)) hide)
+    )
+    (property "LCSC" "C7420346" (at 110.49 118.11 0)
       (effects (font (size 1.27 1.27)) hide)
     )
@@
       (effects (font (size 1.27 1.27)) hide)
     )
+    (property "LCSC" "C25076" (at 93.98 118.11 0)
+      (effects (font (size 1.27 1.27)) hide)
+    )
     (pin "2")
     (pin "1")
@@
       (effects (font (size 1.27 1.27)) (justify right))
     )
-    (property "Footprint" "Diode_SMD:D_SOD-123F" (at 96.52 85.09 0)
+    (property "Footprint" "Diode_SMD:D_SMA" (at 96.52 85.09 0)
       (effects (font (size 1.27 1.27)) hide)
     )
     (property "Datasheet" "~" (at 96.52 85.09 0)
+      (effects (font (size 1.27 1.27)) hide)
+    )
+    (property "LCSC" "C19077489" (at 96.52 85.09 0)
       (effects (font (size 1.27 1.27)) hide)
     )
@@
       (effects (font (size 1.27 1.27)) (justify right))
     )
-    (property "Footprint" "LED_SMD:LED_0603_1608Metric_Pad1.05x0.95mm_HandSolder" (at 74.93 81.28 0)
+    (property "Footprint" "LED_SMD:LED_0603_1608Metric" (at 74.93 81.28 0)
       (effects (font (size 1.27 1.27)) hide)
     )
     (property "Datasheet" "~" (at 74.93 81.28 0)
+      (effects (font (size 1.27 1.27)) hide)
+    )
+    (property "LCSC" "C2286" (at 74.93 81.28 0)
       (effects (font (size 1.27 1.27)) hide)
     )
@@
       (effects (font (size 1.27 1.27)) hide)
     )
+    (property "LCSC" "C25744" (at 74.93 72.39 0)
+      (effects (font (size 1.27 1.27)) hide)
+    )
     (pin "2")
     (pin "1")
@@
     )
   )
-  (symbol (lib_id "Device:D_Schottky") (at 96.52 72.39 90) (mirror x) (unit 1)
-    (in_bom yes) (on_board yes) (dnp no) (fields_autoplaced)
-    (property "Reference" "D10" (at 93.98 70.8025 90)
-      (effects (font (size 1.27 1.27)) (justify left))
+  (symbol (lib_id "Device:D") (at 96.52 72.39 90) (mirror x) (unit 1)
+    (in_bom yes) (on_board yes) (dnp no)
+    (property "Reference" "D10" (at 90.17 71.12 90)
+      (effects (font (size 1.27 1.27)) (justify right))
     )
-    (property "Value" "D_Schottky" (at 93.98 73.3425 90)
-      (effects (font (size 1.27 1.27)) (justify left))
+    (property "Value" "D" (at 90.17 73.66 90)
+      (effects (font (size 1.27 1.27)) (justify right))
     )
     (property "Footprint" "Diode_SMD:D_SOD-123F" (at 96.52 72.39 0)
@@
       (effects (font (size 1.27 1.27)) hide)
     )
-    (property "LCSC" "C22466347" (at 96.52 72.39 0)
+    (property "LCSC" "C18199085" (at 96.52 72.39 0)
       (effects (font (size 1.27 1.27)) hide)
     )
+    (property "Sim.Device" "D" (at 96.52 72.39 0)
+      (effects (font (size 1.27 1.27)) hide)
+    )
+    (property "Sim.Pins" "1=K 2=A" (at 96.52 72.39 0)
+      (effects (font (size 1.27 1.27)) hide)
+    )
