File: STM32F103.kicad_sch (KiCad schematic)
At the start: 14 parts, among them SW4 SW_SPST, U2 STM32F103CBTx, Y1 12MHz

Commit message: add footprint
Changed lines of the file:
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@@
     (stroke (width 0) (type default))
   )
-  (wire (pts (xy 45.72 90.17) (xy 45.72 95.25))
+  (wire (pts (xy 45.72 90.17) (xy 45.72 100.33))
     (stroke (width 0) (type default))
   )
@@
   (wire (pts (xy 118.11 69.85) (xy 118.11 58.42))
     (stroke (width 0) (type default))
+  )
+  (hierarchical_label "GND" (shape output) (at 52.07 121.92 270) (fields_autoplaced)
+    (effects (font (size 1.27 1.27)) (justify right))
+  )
+  (hierarchical_label "GND" (shape output) (at 110.49 153.67 270) (fields_autoplaced)
+    (effects (font (size 1.27 1.27)) (justify right))
+  )
+  (hierarchical_label "GND" (shape output) (at 195.58 40.64 270) (fields_autoplaced)
+    (effects (font (size 1.27 1.27)) (justify right))
   )
   (hierarchical_label "PWR_IN" (shape input) (at 153.67 24.13 90) (fields_autoplaced)
@@
     (effects (font (size 1.27 1.27)) (justify left))
   )
+  (hierarchical_label "GND" (shape output) (at 45.72 100.33 270) (fields_autoplaced)
+    (effects (font (size 1.27 1.27)) (justify right))
+  )
   (hierarchical_label "MCU_run" (shape output) (at 95.25 118.11 180) (fields_autoplaced)
     (effects (font (size 1.27 1.27)) (justify right))
@@
     (effects (font (size 1.27 1.27)) (justify left))
   )
+  (hierarchical_label "GND" (shape output) (at 29.21 100.33 270) (fields_autoplaced)
+    (effects (font (size 1.27 1.27)) (justify right))
+  )
   (hierarchical_label "CAN_TX" (shape output) (at 128.27 105.41 0) (fields_autoplaced)
     (effects (font (size 1.27 1.27)) (justify left))
@@
   )
   (hierarchical_label "EMS_Observe" (shape input) (at 95.25 115.57 180) (fields_autoplaced)
+    (effects (font (size 1.27 1.27)) (justify right))
+  )
+  (hierarchical_label "GND" (shape output) (at 163.83 63.5 270) (fields_autoplaced)
     (effects (font (size 1.27 1.27)) (justify right))
   )
@@
     )
   )
-  (symbol (lib_id "power:GND") (at 195.58 40.64 0) (unit 1)
-    (in_bom yes) (on_board yes) (dnp no) (fields_autoplaced)
-    (property "Reference" "#PWR039" (at 195.58 46.99 0)
-      (effects (font (size 1.27 1.27)) hide)
-    )
-    (property "Value" "GND" (at 195.58 45.72 0)
-      (effects (font (size 1.27 1.27)))
-    )
-    (property "Footprint" "" (at 195.58 40.64 0)
-      (effects (font (size 1.27 1.27)) hide)
-    )
-    (property "Datasheet" "" (at 195.58 40.64 0)
-      (effects (font (size 1.27 1.27)) hide)
-    )
-    (pin "1")
-    (instances
-      (project "schematic_PWRcutoff"
-        (path "/9e89b938-308a-42c1-b814-ac47b1ea682c/7e11ad9c-6cdf-420a-85ee-4145fdfc2616"
-          (reference "#PWR039") (unit 1)
-        )
-      )
-      (project "schematic_PWR"
-        (path "/f4729e9b-1fa3-4d29-bc6f-94f153418360/f20d4b20-da89-4eb5-9739-91620722d466"
-          (reference "#PWR039") (unit 1)
-        )
-      )
-    )
-  )
-  (symbol (lib_id "power:GND") (at 29.21 100.33 0) (unit 1)
-    (in_bom yes) (on_board yes) (dnp no) (fields_autoplaced)
-    (property "Reference" "#PWR033" (at 29.21 106.68 0)
-      (effects (font (size 1.27 1.27)) hide)
-    )
-    (property "Value" "GND" (at 29.21 105.41 0)
-      (effects (font (size 1.27 1.27)))
-    )
-    (property "Footprint" "" (at 29.21 100.33 0)
-      (effects (font (size 1.27 1.27)) hide)
-    )
-    (property "Datasheet" "" (at 29.21 100.33 0)
-      (effects (font (size 1.27 1.27)) hide)
-    )
-    (pin "1")
-    (instances
-      (project "schematic_PWRcutoff"
-        (path "/9e89b938-308a-42c1-b814-ac47b1ea682c/7e11ad9c-6cdf-420a-85ee-4145fdfc2616"
-          (reference "#PWR033") (unit 1)
-        )
-      )
-      (project "schematic_PWR"
-        (path "/f4729e9b-1fa3-4d29-bc6f-94f153418360/f20d4b20-da89-4eb5-9739-91620722d466"
-          (reference "#PWR033") (unit 1)
-        )
-      )
-    )
-  )
-  (symbol (lib_id "power:GND") (at 110.49 153.67 0) (unit 1)
-    (in_bom yes) (on_board yes) (dnp no) (fields_autoplaced)
-    (property "Reference" "#PWR037" (at 110.49 160.02 0)
-      (effects (font (size 1.27 1.27)) hide)
-    )
-    (property "Value" "GND" (at 110.49 158.75 0)
-      (effects (font (size 1.27 1.27)))
-    )
-    (property "Footprint" "" (at 110.49 153.67 0)
-      (effects (font (size 1.27 1.27)) hide)
-    )
-    (property "Datasheet" "" (at 110.49 153.67 0)
-      (effects (font (size 1.27 1.27)) hide)
-    )
-    (pin "1")
-    (instances
-      (project "schematic_PWRcutoff"
-        (path "/9e89b938-308a-42c1-b814-ac47b1ea682c/7e11ad9c-6cdf-420a-85ee-4145fdfc2616"
-          (reference "#PWR037") (unit 1)
-        )
-      )
-      (project "schematic_PWR"
-        (path "/f4729e9b-1fa3-4d29-bc6f-94f153418360/f20d4b20-da89-4eb5-9739-91620722d466"
-          (reference "#PWR037") (unit 1)
-        )
-      )
-    )
-  )
-  (symbol (lib_id "power:GND") (at 52.07 121.92 0) (unit 1)
-    (in_bom yes) (on_board yes) (dnp no) (fields_autoplaced)
-    (property "Reference" "#PWR035" (at 52.07 128.27 0)
-      (effects (font (size 1.27 1.27)) hide)
-    )
-    (property "Value" "GND" (at 52.07 127 0)
-      (effects (font (size 1.27 1.27)))
-    )
-    (property "Footprint" "" (at 52.07 121.92 0)
-      (effects (font (size 1.27 1.27)) hide)
-    )
-    (property "Datasheet" "" (at 52.07 121.92 0)
-      (effects (font (size 1.27 1.27)) hide)
-    )
-    (pin "1")
-    (instances
-      (project "schematic_PWRcutoff"
-        (path "/9e89b938-308a-42c1-b814-ac47b1ea682c/7e11ad9c-6cdf-420a-85ee-4145fdfc2616"
-          (reference "#PWR035") (unit 1)
-        )
-      )
-      (project "schematic_PWR"
-        (path "/f4729e9b-1fa3-4d29-bc6f-94f153418360/f20d4b20-da89-4eb5-9739-91620722d466"
-          (reference "#PWR035") (unit 1)
-        )
-      )
-    )
-  )
   (symbol (lib_id "Device:C_Small") (at 173.99 33.02 0) (unit 1)
     (in_bom yes) (on_board yes) (dnp no) (fields_autoplaced)
@@
         (path "/f4729e9b-1fa3-4d29-bc6f-94f153418360/f20d4b20-da89-4eb5-9739-91620722d466"
           (reference "C8") (unit 1)
-        )
-      )
-    )
-  )
-  (symbol (lib_id "power:GND") (at 45.72 95.25 0) (unit 1)
-    (in_bom yes) (on_board yes) (dnp no) (fields_autoplaced)
-    (property "Reference" "#PWR034" (at 45.72 101.6 0)
-      (effects (font (size 1.27 1.27)) hide)
-    )
-    (property "Value" "GND" (at 45.72 100.33 0)
-      (effects (font (size 1.27 1.27)))
-    )
-    (property "Footprint" "" (at 45.72 95.25 0)
-      (effects (font (size 1.27 1.27)) hide)
-    )
-    (property "Datasheet" "" (at 45.72 95.25 0)
-      (effects (font (size 1.27 1.27)) hide)
-    )
-    (pin "1")
-    (instances
-      (project "schematic_PWRcutoff"
-        (path "/9e89b938-308a-42c1-b814-ac47b1ea682c/7e11ad9c-6cdf-420a-85ee-4145fdfc2616"
-          (reference "#PWR034") (unit 1)
-        )
-      )
-      (project "schematic_PWR"
-        (path "/f4729e9b-1fa3-4d29-bc6f-94f153418360/f20d4b20-da89-4eb5-9739-91620722d466"
-          (reference "#PWR034") (unit 1)
         )
       )
@@
         )
       )
-    )
-  )
-  (symbol (lib_id "power:GND") (at 163.83 63.5 0) (unit 1)
-    (in_bom yes) (on_board yes) (dnp no) (fields_autoplaced)
-    (property "Reference" "#PWR044" (at 163.83 69.85 0)
-      (effects (font (size 1.27 1.27)) hide)
-    )
-    (property "Value" "GND" (at 163.83 68.58 0)
-      (effects (font (size 1.27 1.27)))
-    )
-    (property "Footprint" "" (at 163.83 63.5 0)
-      (effects (font (size 1.27 1.27)) hide)
-    )
-    (property "Datasheet" "" (at 163.83 63.5 0)
-      (effects (font (size 1.27 1.27)) hide)
-    )
-    (pin "1")
-    (instances
-      (project "schematic_PWRcutoff"
-        (path "/9e89b938-308a-42c1-b814-ac47b1ea682c/7e11ad9c-6cdf-420a-85ee-4145fdfc2616"
-          (reference "#PWR044") (unit 1)
-        )
-      )
-      (project "schematic_PWR"
-        (path "/f4729e9b-1fa3-4d29-bc6f-94f153418360/f20d4b20-da89-4eb5-9739-91620722d466"
-          (reference "#PWR044") (unit 1)
-        )
-      )

Commit message: Parts layout finish
Parts:
- C10, C13, C17, C4, C8, C9: footprint Capacitor_SMD:C_0603_1608Metric_Pad1.08x0.95mm_HandSolder -> Capacitor_SMD:C_0402_1005Metric
- C16, C7: footprint Capacitor_SMD:C_0603_1608Metric_Pad1.08x0.95mm_HandSolder -> Capacitor_SMD:C_0603_1608Metric
- C5, C6: value 10pF -> 15pF; footprint Capacitor_SMD:C_0603_1608Metric_Pad1.08x0.95mm_HandSolder -> Capacitor_SMD:C_0402_1005Metric
- R12: footprint Resistor_SMD:R_0603_1608Metric_Pad0.98x0.95mm_HandSolder -> Resistor_SMD:R_0402_1005Metric
- Y1: footprint Crystal:Crystal_SMD_SeikoEpson_FA238V-4Pin_3.2x2.5mm -> Crystal:Crystal_SMD_3225-4Pin_3.2x2.5mm; LCSC (none) -> C9002
Changed lines of the file:
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@@
       (project "schematic_PWR"
         (path "/f4729e9b-1fa3-4d29-bc6f-94f153418360/f20d4b20-da89-4eb5-9739-91620722d466"
-          (reference "SW4") (unit 1)
+          (reference "SW3") (unit 1)
         )
       )
@@
       (effects (font (size 1.27 1.27)) (justify left))
     )
-    (property "Footprint" "Resistor_SMD:R_0603_1608Metric_Pad0.98x0.95mm_HandSolder" (at 43.942 86.36 90)
+    (property "Footprint" "Resistor_SMD:R_0402_1005Metric" (at 43.942 86.36 90)
       (effects (font (size 1.27 1.27)) hide)
     )
@@
       (project "schematic_PWR"
         (path "/f4729e9b-1fa3-4d29-bc6f-94f153418360/f20d4b20-da89-4eb5-9739-91620722d466"
-          (reference "R12") (unit 1)
+          (reference "R18") (unit 1)
         )
       )
@@
       (project "schematic_PWR"
         (path "/f4729e9b-1fa3-4d29-bc6f-94f153418360/f20d4b20-da89-4eb5-9739-91620722d466"
-          (reference "#PWR036") (unit 1)
+          (reference "#PWR040") (unit 1)
         )
       )
@@
       (project "schematic_PWR"
         (path "/f4729e9b-1fa3-4d29-bc6f-94f153418360/f20d4b20-da89-4eb5-9739-91620722d466"
-          (reference "U2") (unit 1)
+          (reference "U3") (unit 1)
         )
       )
@@
       (effects (font (size 1.27 1.27)) (justify left))
     )
-    (property "Footprint" "Capacitor_SMD:C_0603_1608Metric_Pad1.08x0.95mm_HandSolder" (at 184.15 33.02 0)
+    (property "Footprint" "Capacitor_SMD:C_0402_1005Metric" (at 184.15 33.02 0)
       (effects (font (size 1.27 1.27)) hide)
     )
@@
       (project "schematic_PWR"
         (path "/f4729e9b-1fa3-4d29-bc6f-94f153418360/f20d4b20-da89-4eb5-9739-91620722d466"
-          (reference "C10") (unit 1)
+          (reference "C26") (unit 1)
         )
       )
@@
       (effects (font (size 1.27 1.27)) (justify left))
     )
-    (property "Footprint" "Capacitor_SMD:C_0603_1608Metric_Pad1.08x0.95mm_HandSolder" (at 173.99 33.02 0)
+    (property "Footprint" "Capacitor_SMD:C_0402_1005Metric" (at 173.99 33.02 0)
       (effects (font (size 1.27 1.27)) hide)
     )
@@
       (project "schematic_PWR"
         (path "/f4729e9b-1fa3-4d29-bc6f-94f153418360/f20d4b20-da89-4eb5-9739-91620722d466"
-          (reference "C9") (unit 1)
+          (reference "C25") (unit 1)
         )
       )
@@
       (effects (font (size 1.27 1.27)) (justify left))
     )
-    (property "Footprint" "Capacitor_SMD:C_0603_1608Metric_Pad1.08x0.95mm_HandSolder" (at 195.58 33.02 0)
+    (property "Footprint" "Capacitor_SMD:C_0402_1005Metric" (at 195.58 33.02 0)
       (effects (font (size 1.27 1.27)) hide)
     )
@@
       (project "schematic_PWR"
         (path "/f4729e9b-1fa3-4d29-bc6f-94f153418360/f20d4b20-da89-4eb5-9739-91620722d466"
-          (reference "C13") (unit 1)
+          (reference "C27") (unit 1)
         )
       )
@@
       (effects (font (size 1.27 1.27)) (justify left))
     )
-    (property "Footprint" "Capacitor_SMD:C_0603_1608Metric_Pad1.08x0.95mm_HandSolder" (at 163.83 55.88 0)
+    (property "Footprint" "Capacitor_SMD:C_0402_1005Metric" (at 163.83 55.88 0)
       (effects (font (size 1.27 1.27)) hide)
     )
@@
       (project "schematic_PWR"
         (path "/f4729e9b-1fa3-4d29-bc6f-94f153418360/f20d4b20-da89-4eb5-9739-91620722d466"
-          (reference "C17") (unit 1)
+          (reference "C24") (unit 1)
         )
       )
@@
       (effects (font (size 1.27 1.27)) (justify left))
     )
-    (property "Footprint" "Capacitor_SMD:C_0603_1608Metric_Pad1.08x0.95mm_HandSolder" (at 35.56 86.36 0)
+    (property "Footprint" "Capacitor_SMD:C_0402_1005Metric" (at 35.56 86.36 0)
       (effects (font (size 1.27 1.27)) hide)
     )
@@
       (project "schematic_PWR"
         (path "/f4729e9b-1fa3-4d29-bc6f-94f153418360/f20d4b20-da89-4eb5-9739-91620722d466"
-          (reference "C4") (unit 1)
+          (reference "C18") (unit 1)
         )
       )
@@
       (effects (font (size 1.27 1.27)) (justify left))
     )
-    (property "Footprint" "Capacitor_SMD:C_0603_1608Metric_Pad1.08x0.95mm_HandSolder" (at 163.83 33.02 0)
+    (property "Footprint" "Capacitor_SMD:C_0402_1005Metric" (at 163.83 33.02 0)
       (effects (font (size 1.27 1.27)) hide)
     )
@@
       (project "schematic_PWR"
         (path "/f4729e9b-1fa3-4d29-bc6f-94f153418360/f20d4b20-da89-4eb5-9739-91620722d466"
-          (reference "C8") (unit 1)
+          (reference "C23") (unit 1)
         )
       )
@@
       (effects (font (size 1.27 1.27)) (justify left))
     )
-    (property "Value" "10pF" (at 58.42 114.3063 0)
-      (effects (font (size 1.27 1.27)) (justify left))
-    )
-    (property "Footprint" "Capacitor_SMD:C_0603_1608Metric_Pad1.08x0.95mm_HandSolder" (at 55.88 113.03 0)
+    (property "Value" "15pF" (at 58.42 114.3063 0)
+      (effects (font (size 1.27 1.27)) (justify left))
+    )
+    (property "Footprint" "Capacitor_SMD:C_0402_1005Metric" (at 55.88 113.03 0)
       (effects (font (size 1.27 1.27)) hide)
     )
@@
       (project "schematic_PWR"
         (path "/f4729e9b-1fa3-4d29-bc6f-94f153418360/f20d4b20-da89-4eb5-9739-91620722d466"
-          (reference "C5") (unit 1)
+          (reference "C19") (unit 1)
         )
       )
@@
       (project "schematic_PWR"
         (path "/f4729e9b-1fa3-4d29-bc6f-94f153418360/f20d4b20-da89-4eb5-9739-91620722d466"
-          (reference "#PWR038") (unit 1)
+          (reference "#PWR043") (unit 1)
         )
       )
@@
       (effects (font (size 1.27 1.27)))
     )
-    (property "Footprint" "Crystal:Crystal_SMD_SeikoEpson_FA238V-4Pin_3.2x2.5mm" (at 62.23 99.06 0)
+    (property "Footprint" "Crystal:Crystal_SMD_3225-4Pin_3.2x2.5mm" (at 62.23 99.06 0)
       (effects (font (size 1.27 1.27)) hide)
     )
@@
     )
     (property "name" "" (at 62.23 99.06 0)
+      (effects (font (size 1.27 1.27)) hide)
+    )
+    (property "LCSC" "C9002" (at 62.23 99.06 0)
       (effects (font (size 1.27 1.27)) hide)
     )
@@
       (effects (font (size 1.27 1.27)) (justify left))
     )
-    (property "Footprint" "Capacitor_SMD:C_0603_1608Metric_Pad1.08x0.95mm_HandSolder" (at 153.67 55.88 0)
+    (property "Footprint" "Capacitor_SMD:C_0603_1608Metric" (at 153.67 55.88 0)
       (effects (font (size 1.27 1.27)) hide)
     )
@@
       (project "schematic_PWR"
         (path "/f4729e9b-1fa3-4d29-bc6f-94f153418360/f20d4b20-da89-4eb5-9739-91620722d466"
-          (reference "C16") (unit 1)
+          (reference "C22") (unit 1)
         )
       )
@@
       (effects (font (size 1.27 1.27)) (justify left))
     )
-    (property "Footprint" "Capacitor_SMD:C_0603_1608Metric_Pad1.08x0.95mm_HandSolder" (at 153.67 33.02 0)
+    (property "Footprint" "Capacitor_SMD:C_0603_1608Metric" (at 153.67 33.02 0)
       (effects (font (size 1.27 1.27)) hide)
     )
@@
       (project "schematic_PWR"
         (path "/f4729e9b-1fa3-4d29-bc6f-94f153418360/f20d4b20-da89-4eb5-9739-91620722d466"
-          (reference "C7") (unit 1)
+          (reference "C21") (unit 1)
         )
       )
@@
       (effects (font (size 1.27 1.27)) (justify left))
     )
-    (property "Value" "10pF" (at 69.85 114.3063 0)
-      (effects (font (size 1.27 1.27)) (justify left))
-    )
-    (property "Footprint" "Capacitor_SMD:C_0603_1608Metric_Pad1.08x0.95mm_HandSolder" (at 67.31 113.03 0)
+    (property "Value" "15pF" (at 69.85 114.3063 0)
+      (effects (font (size 1.27 1.27)) (justify left))
+    )
+    (property "Footprint" "Capacitor_SMD:C_0402_1005Metric" (at 67.31 113.03 0)
       (effects (font (size 1.27 1.27)) hide)
     )
@@
       (project "schematic_PWR"
         (path "/f4729e9b-1fa3-4d29-bc6f-94f153418360/f20d4b20-da89-4eb5-9739-91620722d466"
-          (reference "C6") (unit 1)
+          (reference "C20") (unit 1)
         )
       )
@@
       (project "schematic_PWR"
         (path "/f4729e9b-1fa3-4d29-bc6f-94f153418360/f20d4b20-da89-4eb5-9739-91620722d466"
-          (reference "#PWR043") (unit 1)
+          (reference "#PWR041") (unit 1)
         )
       )
@@
       (project "schematic_PWR"
         (path "/f4729e9b-1fa3-4d29-bc6f-94f153418360/f20d4b20-da89-4eb5-9739-91620722d466"
-          (reference "#PWR045") (unit 1)
-        )
-      )
+          (reference "#PWR042") (unit 1)
+        )
+      )

Commit message: アートワークのほとんど終わり
Parts:
- C10, C13, C17, C4, C8, C9: LCSC (none) -> C307331
- C16, C7: LCSC (none) -> C19702
- C5, C6: LCSC (none) -> C1548
- R12: LCSC (none) -> C25744
- SW4: footprint Button_Switch_THT:SW_PUSH_6mm_H7.3mm -> RDC_generic:TVBP06-B043
- U2: LCSC (none) -> C8734
Connections:
- net EMS_Observe: now also U2.19 (PB1); no longer U2.41 (PB5)
- net EMS_Signal: now also U2.18 (PB0); no longer U2.40 (PB4)
- net MCU_run: now also U2.17 (PA7); no longer U2.42 (PB6)
Changed lines of the file:
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@@
   (junction (at 67.31 99.06) (diameter 0) (color 0 0 0 0)
   )
-  (no_connect (at 95.25 102.87))
   (no_connect (at 128.27 77.47))
   (no_connect (at 95.25 123.19))
@@
   (no_connect (at 95.25 97.79))
   (no_connect (at 95.25 128.27))
+  (no_connect (at 95.25 115.57))
   (no_connect (at 128.27 80.01))
   (no_connect (at 128.27 97.79))
-  (no_connect (at 95.25 105.41))
   (no_connect (at 128.27 87.63))
-  (no_connect (at 95.25 107.95))
   (no_connect (at 95.25 135.89))
   (no_connect (at 95.25 92.71))
@@
   (no_connect (at 128.27 90.17))
   (no_connect (at 95.25 140.97))
+  (no_connect (at 95.25 113.03))
   (no_connect (at 95.25 130.81))
   (no_connect (at 128.27 95.25))
-  (no_connect (at 128.27 92.71))
   (no_connect (at 95.25 138.43))
   (no_connect (at 128.27 85.09))
   (no_connect (at 95.25 133.35))
+  (no_connect (at 95.25 107.95))
+  (no_connect (at 95.25 118.11))
   (wire (pts (xy 184.15 27.94) (xy 195.58 27.94))
     (stroke (width 0) (type default))
@@
   (wire (pts (xy 118.11 69.85) (xy 118.11 58.42))
     (stroke (width 0) (type default))
+  )
+  (hierarchical_label "EMS_Signal" (shape output) (at 95.25 102.87 180) (fields_autoplaced)
+    (effects (font (size 1.27 1.27)) (justify right))
   )
   (hierarchical_label "GND" (shape output) (at 52.07 121.92 270) (fields_autoplaced)
@@
     (effects (font (size 1.27 1.27)) (justify right))
   )
-  (hierarchical_label "MCU_run" (shape output) (at 95.25 118.11 180) (fields_autoplaced)
-    (effects (font (size 1.27 1.27)) (justify right))
-  )
   (hierarchical_label "PWR_IN" (shape input) (at 153.67 48.26 90) (fields_autoplaced)
     (effects (font (size 1.27 1.27)) (justify left))
@@
     (effects (font (size 1.27 1.27)) (justify left))
   )
-  (hierarchical_label "EMS_Signal" (shape output) (at 95.25 113.03 180) (fields_autoplaced)
-    (effects (font (size 1.27 1.27)) (justify right))
-  )
   (hierarchical_label "SWDIO" (shape bidirectional) (at 128.27 107.95 0) (fields_autoplaced)
     (effects (font (size 1.27 1.27)) (justify left))
   )
+  (hierarchical_label "MCU_run" (shape output) (at 128.27 92.71 0) (fields_autoplaced)
+    (effects (font (size 1.27 1.27)) (justify left))
+  )
   (hierarchical_label "SWO" (shape bidirectional) (at 95.25 110.49 180) (fields_autoplaced)
     (effects (font (size 1.27 1.27)) (justify right))
   )
-  (hierarchical_label "EMS_Observe" (shape input) (at 95.25 115.57 180) (fields_autoplaced)
+  (hierarchical_label "GND" (shape output) (at 163.83 63.5 270) (fields_autoplaced)
     (effects (font (size 1.27 1.27)) (justify right))
   )
-  (hierarchical_label "GND" (shape output) (at 163.83 63.5 270) (fields_autoplaced)
+  (hierarchical_label "EMS_Observe" (shape input) (at 95.25 105.41 180) (fields_autoplaced)
     (effects (font (size 1.27 1.27)) (justify right))
   )
@@
       (effects (font (size 1.27 1.27)) (justify left))
     )
-    (property "Footprint" "Button_Switch_THT:SW_PUSH_6mm_H7.3mm" (at 29.21 86.36 0)
+    (property "Footprint" "RDC_generic:TVBP06-B043" (at 29.21 86.36 0)
       (effects (font (size 1.27 1.27)) hide)
     )
@@
     )
     (property "name" "" (at 45.72 86.36 0)
+      (effects (font (size 1.27 1.27)) hide)
+    )
+    (property "LCSC" "C25744" (at 45.72 86.36 0)
       (effects (font (size 1.27 1.27)) hide)
     )
@@
     )
     (property "name" "" (at 110.49 110.49 0)
+      (effects (font (size 1.27 1.27)) hide)
+    )
+    (property "LCSC" "C8734" (at 110.49 110.49 0)
       (effects (font (size 1.27 1.27)) hide)
     )
@@
       (effects (font (size 1.27 1.27)) hide)
     )
+    (property "LCSC" "C307331" (at 184.15 33.02 0)
+      (effects (font (size 1.27 1.27)) hide)
+    )
     (pin "2")
     (pin "1")
@@
       (effects (font (size 1.27 1.27)) hide)
     )
+    (property "LCSC" "C307331" (at 173.99 33.02 0)
+      (effects (font (size 1.27 1.27)) hide)
+    )
     (pin "2")
     (pin "1")
@@
       (effects (font (size 1.27 1.27)) hide)
     )
+    (property "LCSC" "C307331" (at 195.58 33.02 0)
+      (effects (font (size 1.27 1.27)) hide)
+    )
     (pin "2")
     (pin "1")
@@
       (effects (font (size 1.27 1.27)) hide)
     )
+    (property "LCSC" "C307331" (at 163.83 55.88 0)
+      (effects (font (size 1.27 1.27)) hide)
+    )
     (pin "2")
     (pin "1")
@@
       (effects (font (size 1.27 1.27)) hide)
     )
+    (property "LCSC" "C307331" (at 35.56 86.36 0)
+      (effects (font (size 1.27 1.27)) hide)
+    )
     (pin "2")
     (pin "1")
@@
       (effects (font (size 1.27 1.27)) hide)
     )
+    (property "LCSC" "C307331" (at 163.83 33.02 0)
+      (effects (font (size 1.27 1.27)) hide)
+    )
     (pin "2")
     (pin "1")
@@
     )
     (property "name" "" (at 55.88 113.03 0)
+      (effects (font (size 1.27 1.27)) hide)
+    )
+    (property "LCSC" "C1548" (at 55.88 113.03 0)
       (effects (font (size 1.27 1.27)) hide)
     )
@@
       (effects (font (size 1.27 1.27)) hide)
     )
+    (property "LCSC" "C19702" (at 153.67 55.88 0)
+      (effects (font (size 1.27 1.27)) hide)
+    )
     (pin "2")
     (pin "1")
@@
       (effects (font (size 1.27 1.27)) hide)
     )
+    (property "LCSC" "C19702" (at 153.67 33.02 0)
+      (effects (font (size 1.27 1.27)) hide)
+    )
     (pin "2")
     (pin "1")
@@
       (effects (font (size 1.27 1.27)) hide)
     )
+    (property "LCSC" "C1548" (at 67.31 113.03 0)
+      (effects (font (size 1.27 1.27)) hide)
+    )
