File: Stepdown_12V_8A.kicad_sch (KiCad schematic)
At the start: 16 parts

Commit message: Parts layout finish
Parts:
- added D6: D_Zener, Diode_SMD:D_SOD-123F, symbol Device:D_Zener
- added R1 (x2): 10k, Resistor_SMD:R_0402_1005Metric, symbol Device:R_Small
- C1, C2, C3, C4, C6: footprint (none) -> Capacitor_SMD:C_0603_1608Metric
- C10, C5, C7, C8, C9: footprint (none) -> Capacitor_SMD:C_1210_3225Metric
- L1: value 2.2u -> 8.2u; footprint (none) -> Inductor_SMD:L_Sunlord_MWSA1004S; LCSC (none) -> C167232
- R1: value 105k -> 205k; footprint (none) -> Resistor_SMD:R_0402_1005Metric
- R2, R3, R4: footprint (none) -> Resistor_SMD:R_0402_1005Metric
- U1: value ~ -> XR76208; LCSC (none) -> C555356
Connections:
- net Vin: now also R1.1
- net GND: now reaches C5.2, C7.2, C8.2
- net GND: now also C1.2, C10.2, C2.2, C6.2, C9.2, R1.2, R4.2, U1.10 (AGND), U1.15 (PGND), U1.16 (PGND), U1.17 (PGND), U1.18 (PGND), U1.19 (PGND), U1.7 (AGND), U1.AGND, U1.PGND, D6.2 (A)
- net at U1.2 (EN/MODE): now also D6.1 (K), R1.2
- net at U1.5 (P_{GOOD}): now also R1.1
- net at C6.1, U1.9 (V_{CC}): now also R1.2
Other:
- moved on the sheet: C1, C10, C9

Commit message: アートワークのほとんど終わり
Parts:
- C1: LCSC (none) -> C14663
- C10, C9: LCSC (none) -> C337485
- C2: LCSC (none) -> C1622
- C3: LCSC (none) -> C15849
- C4: LCSC (none) -> C28262
- C5, C7, C8: LCSC (none) -> C90142
- C6: LCSC (none) -> C1779
- D6: footprint Diode_SMD:D_SOD-123F -> Diode_SMD:D_SOD-123; LCSC (none) -> C19077392
- L1: value 8.2u -> 8.2uH
- R1: LCSC (none) -> C25744
- R1: LCSC (none) -> C226887
- R2: LCSC (none) -> C25900
- R3: value 38k -> 47k; LCSC (none) -> C25792
- R4: value 2k -> 2.4k; LCSC (none) -> C25882
Connections:
- net at C3.1, L1.1, R2.1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: no longer U1.20 (SW)
Changed lines of the file:
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@@
+      (effects (font (size 1.27 1.27)) hide)
+    )
+    (property "LCSC" "C90142" (at 219.71 74.93 0)
       (effects (font (size 1.27 1.27)) hide)
     )
@@
       (effects (font (size 1.27 1.27)) hide)
     )
+    (property "LCSC" "C90142" (at 209.55 74.93 0)
+      (effects (font (size 1.27 1.27)) hide)
+    )
     (pin "2")
     (pin "1")
@@
       (effects (font (size 1.27 1.27)) hide)
     )
+    (property "LCSC" "C90142" (at 199.39 74.93 0)
+      (effects (font (size 1.27 1.27)) hide)
+    )
     (pin "2")
     (pin "1")
@@
       (effects (font (size 1.27 1.27)) hide)
     )
+    (property "LCSC" "C25744" (at 82.55 60.96 0)
+      (effects (font (size 1.27 1.27)) hide)
+    )
     (pin "1")
     (pin "2")
@@
       (effects (font (size 1.27 1.27)) (justify right))
     )
-    (property "Value" "2k" (at 187.96 82.55 0)
+    (property "Value" "2.4k" (at 187.96 82.55 0)
       (effects (font (size 1.27 1.27)) (justify right))
     )
@@
       (effects (font (size 1.27 1.27)) hide)
     )
+    (property "LCSC" "C25882" (at 185.42 81.28 0)
+      (effects (font (size 1.27 1.27)) hide)
+    )
     (pin "1")
     (pin "2")
@@
     )
     (property "Datasheet" "~" (at 111.76 73.66 0)
+      (effects (font (size 1.27 1.27)) hide)
+    )
+    (property "LCSC" "C1622" (at 111.76 73.66 0)
       (effects (font (size 1.27 1.27)) hide)
     )
@@
       (effects (font (size 1.27 1.27)) hide)
     )
+    (property "LCSC" "C25900" (at 152.4 69.85 0)
+      (effects (font (size 1.27 1.27)) hide)
+    )
     (pin "1")
     (pin "2")
@@
       (effects (font (size 1.27 1.27)) hide)
     )
+    (property "LCSC" "C337485" (at 36.83 64.77 0)
+      (effects (font (size 1.27 1.27)) hide)
+    )
     (pin "2")
     (pin "1")
@@
       (effects (font (size 1.27 1.27)) hide)
     )
+    (property "LCSC" "C226887" (at 119.38 78.74 0)
+      (effects (font (size 1.27 1.27)) hide)
+    )
     (pin "1")
     (pin "2")
@@
       (effects (font (size 1.27 1.27)) (justify right))
     )
-    (property "Footprint" "Diode_SMD:D_SOD-123F" (at 82.55 72.39 0)
+    (property "Footprint" "Diode_SMD:D_SOD-123" (at 82.55 72.39 0)
       (effects (font (size 1.27 1.27)) hide)
     )
@@
       (effects (font (size 1.27 1.27)) hide)
     )
+    (property "LCSC" "C19077392" (at 82.55 72.39 0)
+      (effects (font (size 1.27 1.27)) hide)
+    )
     (pin "1")
     (pin "2")
@@
       (effects (font (size 1.27 1.27)) (justify right))
     )
-    (property "Value" "38k" (at 187.96 72.39 0)
+    (property "Value" "47k" (at 187.96 72.39 0)
       (effects (font (size 1.27 1.27)) (justify right))
     )
@@
       (effects (font (size 1.27 1.27)) hide)
     )
+    (property "LCSC" "C25792" (at 185.42 71.12 0)
+      (effects (font (size 1.27 1.27)) hide)
+    )
     (pin "1")
     (pin "2")
@@
     )
     (property "Datasheet" "~" (at 101.6 63.5 0)
+      (effects (font (size 1.27 1.27)) hide)
+    )
+    (property "LCSC" "C25744" (at 101.6 63.5 0)
       (effects (font (size 1.27 1.27)) hide)
     )
@@
       (effects (font (size 1.27 1.27)))
     )
-    (property "Value" "8.2u" (at 172.72 59.69 90)
+    (property "Value" "8.2uH" (at 172.72 59.69 90)
       (effects (font (size 1.27 1.27)))
     )
@@
       (effects (font (size 1.27 1.27)) hide)
     )
+    (property "LCSC" "C15849" (at 152.4 58.42 0)
+      (effects (font (size 1.27 1.27)) hide)
+    )
     (pin "2")
     (pin "1")
@@
       (effects (font (size 1.27 1.27)) hide)
     )
+    (property "LCSC" "C28262" (at 180.34 71.12 0)
+      (effects (font (size 1.27 1.27)) hide)
+    )
     (pin "2")
     (pin "1")
@@
       (effects (font (size 1.27 1.27)) hide)
     )
+    (property "LCSC" "C14663" (at 58.42 64.77 0)
+      (effects (font (size 1.27 1.27)) hide)
+    )
     (pin "2")
     (pin "1")
@@
       (effects (font (size 1.27 1.27)) hide)
     )
+    (property "LCSC" "C337485" (at 46.99 64.77 0)
+      (effects (font (size 1.27 1.27)) hide)
+    )
     (pin "2")
     (pin "1")
@@
       (effects (font (size 1.27 1.27)) hide)
     )
+    (property "LCSC" "C1779" (at 101.6 73.66 0)
+      (effects (font (size 1.27 1.27)) hide)
+    )
